Commit message: Fix mesh files

File: robots/g1_description/g1_23dof.urdf (robot description, URDF)
Before this commit: robot g1_23dof, 32 links, 31 joints
Links:
- link head_link: geometry collision mesh filename=package:://g1_description/meshes/head_link.STL; visual mesh filename=package:://g1_description/meshes/head_link.STL
- link left_ankle_pitch_link: geometry collision mesh filename=package:://g1_description/meshes/left_ankle_pitch_link.STL; visual mesh filename=package:://g1_description/meshes/left_ankle_pitch_link.STL
- link left_ankle_roll_link: geometry collision sphere radius=0.005; collision sphere radius=0.005
- link left_elbow_link: geometry collision mesh filename=package:://g1_description/meshes/left_elbow_link.STL; visual mesh filename=package:://g1_description/meshes/left_elbow_link.STL
- link left_hip_pitch_link: geometry collision mesh filename=package:://g1_description/meshes/left_hip_pitch_link.STL; visual mesh filename=package:://g1_description/meshes/left_hip_pitch_link.STL
- link left_hip_roll_link: geometry collision mesh filename=package:://g1_description/meshes/left_hip_roll_link.STL; visual mesh filename=package:://g1_description/meshes/left_hip_roll_link.STL
- link left_hip_yaw_link: geometry collision mesh filename=package:://g1_description/meshes/left_hip_yaw_link.STL; visual mesh filename=package:://g1_description/meshes/left_hip_yaw_link.STL
- link left_knee_link: geometry collision mesh filename=package:://g1_description/meshes/left_knee_link.STL; visual mesh filename=package:://g1_description/meshes/left_knee_link.STL
- link left_shoulder_pitch_link: geometry collision cylinder length=0.05 radius=0.03; visual mesh filename=package:://g1_description/meshes/left_shoulder_pitch_link.S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
- link left_shoulder_roll_link: geometry collision cylinder length=0.03 radius=0.03; visual mesh filename=package:://g1_description/meshes/left_shoulder_roll_link.STL
- link left_shoulder_yaw_link: geometry collision mesh filename=package:://g1_description/meshes/left_shoulder_yaw_link.STL; visual mesh filename=package:://g1_description/meshes/left_shoulder_yaw_link.STL
- link left_wrist_roll_rubber_hand: geometry collision mesh filename=package:://g1_description/meshes/left_wrist_roll_rubber_han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; visual mesh filename=package:://g1_description/meshes/left_wrist_roll_rubber_han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
- link logo_link: geometry collision mesh filename=package:://g1_description/meshes/logo_link.STL; visual mesh filename=package:://g1_description/meshes/logo_link.STL
- link pelvis: geometry visual mesh filename=package:://g1_description/meshes/pelvis.STL
- link pelvis_contour_link: geometry collision mesh filename=package:://g1_description/meshes/pelvis_contour_link.STL; visual mesh filename=package:://g1_description/meshes/pelvis_contour_link.STL
- link right_ankle_pitch_link: geometry collision mesh filename=package:://g1_description/meshes/right_ankle_pitch_link.STL; visual mesh filename=package:://g1_description/meshes/right_ankle_pitch_link.STL
- link right_ankle_roll_link: geometry collision sphere radius=0.005; collision sphere radius=0.005
- link right_elbow_link: geometry collision mesh filename=package:://g1_description/meshes/right_elbow_link.STL; visual mesh filename=package:://g1_description/meshes/right_elbow_link.STL
- link right_hip_pitch_link: geometry collision mesh filename=package:://g1_description/meshes/right_hip_pitch_link.STL; visual mesh filename=package:://g1_description/meshes/right_hip_pitch_link.STL
- link right_hip_roll_link: geometry collision mesh filename=package:://g1_description/meshes/right_hip_roll_link.STL; visual mesh filename=package:://g1_description/meshes/right_hip_roll_link.STL
- link right_hip_yaw_link: geometry collision mesh filename=package:://g1_description/meshes/right_hip_yaw_link.STL; visual mesh filename=package:://g1_description/meshes/right_hip_yaw_link.STL
- link right_knee_link: geometry collision mesh filename=package:://g1_description/meshes/right_knee_link.STL; visual mesh filename=package:://g1_description/meshes/right_knee_link.STL
- link right_shoulder_pitch_link: geometry collision cylinder length=0.05 radius=0.03; visual mesh filename=package:://g1_description/meshes/right_shoulder_pitch_link.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
- link right_shoulder_roll_link: geometry collision cylinder length=0.03 radius=0.03; visual mesh filename=package:://g1_description/meshes/right_shoulder_roll_link.S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
- link right_shoulder_yaw_link: geometry collision mesh filename=package:://g1_description/meshes/right_shoulder_yaw_link.STL; visual mesh filename=package:://g1_description/meshes/right_shoulder_yaw_link.STL
- link right_wrist_roll_rubber_hand: geometry collision mesh filename=package:://g1_description/meshes/right_wrist_roll_rubber_ha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; visual mesh filename=package:://g1_description/meshes/right_wrist_roll_rubber_ha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
- link torso_link: geometry collision mesh filename=package:://g1_description/meshes/torso_link.STL; visual mesh filename=package:://g1_description/meshes/torso_link.STL
- link waist_support_link: geometry collision mesh filename=package:://g1_description/meshes/waist_support_link.STL; visual mesh filename=package:://g1_description/meshes/waist_support_link.STL
- link waist_yaw_fixed_link: geometry visual mesh filename=package:://g1_description/meshes/waist_yaw_link.STL

Commit message: Add contact frames to urdf for plane, line and point contacts

File: robots/g1_description/g1_23dof.urdf (robot description, URDF)
Before this commit: robot g1_23dof, 32 links, 31 joints
Links:
- added link left_foot_line_contact_lower
- added link left_foot_line_contact_upper
- added link left_foot_lower_left
- added link left_foot_lower_right
- added link left_foot_point_contact
- added link left_foot_upper_left
- added link left_foot_upper_right
- added link right_foot_line_contact_lower
- added link right_foot_line_contact_upper
- added link right_foot_lower_left
- added link right_foot_lower_right
- added link right_foot_point_contact
- added link right_foot_upper_left
- added link right_foot_upper_right
- link head_link: geometry collision mesh filename=package://g1_description/meshes/head_link.STL; visual mesh filename=package://g1_description/meshes/head_link.STL
- link left_ankle_pitch_link: geometry collision mesh filename=package://g1_description/meshes/left_ankle_pitch_link.STL; visual mesh filename=package://g1_description/meshes/left_ankle_pitch_link.STL
- link left_ankle_roll_link: geometry collision sphere radius=0.005; collision sphere radius=0.005
- link left_elbow_link: geometry collision mesh filename=package://g1_description/meshes/left_elbow_link.STL; visual mesh filename=package://g1_description/meshes/left_elbow_link.STL
- link left_hip_pitch_link: geometry collision mesh filename=package://g1_description/meshes/left_hip_pitch_link.STL; visual mesh filename=package://g1_description/meshes/left_hip_pitch_link.STL
- link left_hip_roll_link: geometry collision mesh filename=package://g1_description/meshes/left_hip_roll_link.STL; visual mesh filename=package://g1_description/meshes/left_hip_roll_link.STL
- link left_hip_yaw_link: geometry collision mesh filename=package://g1_description/meshes/left_hip_yaw_link.STL; visual mesh filename=package://g1_description/meshes/left_hip_yaw_link.STL
- link left_knee_link: geometry collision mesh filename=package://g1_description/meshes/left_knee_link.STL; visual mesh filename=package://g1_description/meshes/left_knee_link.STL
- link left_shoulder_pitch_link: geometry collision cylinder length=0.05 radius=0.03; visual mesh filename=package://g1_description/meshes/left_shoulder_pitch_link.STL
- link left_shoulder_roll_link: geometry collision cylinder length=0.03 radius=0.03; visual mesh filename=package://g1_description/meshes/left_shoulder_roll_link.STL
- link left_shoulder_yaw_link: geometry collision mesh filename=package://g1_description/meshes/left_shoulder_yaw_link.STL; visual mesh filename=package://g1_description/meshes/left_shoulder_yaw_link.STL
- link left_wrist_roll_rubber_hand: geometry collision mesh filename=package://g1_description/meshes/left_wrist_roll_rubber_hand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; visual mesh filename=package://g1_description/meshes/left_wrist_roll_rubber_hand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
- link logo_link: geometry collision mesh filename=package://g1_description/meshes/logo_link.STL; visual mesh filename=package://g1_description/meshes/logo_link.STL
- link pelvis: geometry visual mesh filename=package://g1_description/meshes/pelvis.STL
- link pelvis_contour_link: geometry collision mesh filename=package://g1_description/meshes/pelvis_contour_link.STL; visual mesh filename=package://g1_description/meshes/pelvis_contour_link.STL
- link right_ankle_pitch_link: geometry collision mesh filename=package://g1_description/meshes/right_ankle_pitch_link.STL; visual mesh filename=package://g1_description/meshes/right_ankle_pitch_link.STL
- link right_ankle_roll_link: geometry collision sphere radius=0.005; collision sphere radius=0.005
- link right_elbow_link: geometry collision mesh filename=package://g1_description/meshes/right_elbow_link.STL; visual mesh filename=package://g1_description/meshes/right_elbow_link.STL
- link right_hip_pitch_link: geometry collision mesh filename=package://g1_description/meshes/right_hip_pitch_link.STL; visual mesh filename=package://g1_description/meshes/right_hip_pitch_link.STL
- link right_hip_roll_link: geometry collision mesh filename=package://g1_description/meshes/right_hip_roll_link.STL; visual mesh filename=package://g1_description/meshes/right_hip_roll_link.STL
- link right_hip_yaw_link: geometry collision mesh filename=package://g1_description/meshes/right_hip_yaw_link.STL; visual mesh filename=package://g1_description/meshes/right_hip_yaw_link.STL
- link right_knee_link: geometry collision mesh filename=package://g1_description/meshes/right_knee_link.STL; visual mesh filename=package://g1_description/meshes/right_knee_link.STL
- link right_shoulder_pitch_link: geometry collision cylinder length=0.05 radius=0.03; visual mesh filename=package://g1_description/meshes/right_shoulder_pitch_link.S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
- link right_shoulder_roll_link: geometry collision cylinder length=0.03 radius=0.03; visual mesh filename=package://g1_description/meshes/right_shoulder_roll_link.STL
- link right_shoulder_yaw_link: geometry collision mesh filename=package://g1_description/meshes/right_shoulder_yaw_link.STL; visual mesh filename=package://g1_description/meshes/right_shoulder_yaw_link.STL
- link right_wrist_roll_rubber_hand: geometry collision mesh filename=package://g1_description/meshes/right_wrist_roll_rubber_han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; visual mesh filename=package://g1_description/meshes/right_wrist_roll_rubber_han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
- link torso_link: geometry collision mesh filename=package://g1_description/meshes/torso_link.STL; visual mesh filename=package://g1_description/meshes/torso_link.STL
- link waist_support_link: geometry collision mesh filename=package://g1_description/meshes/waist_support_link.STL; visual mesh filename=package://g1_description/meshes/waist_support_link.STL
- link waist_yaw_fixed_link: geometry visual mesh filename=package://g1_description/meshes/waist_yaw_link.STL
Joints:
- added joint left_foot_line_contact_lower_fix_joint: type fixed, parent left_ankle_roll_link, child left_foot_line_contact_lower, origin xyz=-0.05 0.0 -0.03 rpy=0 0 0
- added joint left_foot_line_contact_upper_fix_joint: type fixed, parent left_ankle_roll_link, child left_foot_line_contact_upper, origin xyz=0.12 0.0 -0.03 rpy=0 0 0
- added joint left_foot_lower_left_fix_joint: type fixed, parent left_ankle_roll_link, child left_foot_lower_left, origin xyz=-0.05 0.025 -0.03 rpy=0 0 0
- added joint left_foot_lower_right_fix_joint: type fixed, parent left_ankle_roll_link, child left_foot_lower_right, origin xyz=-0.05 -0.025 -0.03 rpy=0 0 0
- added joint left_foot_point_contact_fix_joint: type fixed, parent left_ankle_roll_link, child left_foot_point_contact, origin xyz=0.0 0.0 -0.03 rpy=0 0 0
- added joint left_foot_upper_left_fix_joint: type fixed, parent left_ankle_roll_link, child left_foot_upper_left, origin xyz=0.12 0.03 -0.03 rpy=0 0 0
- added joint left_foot_upper_right_fix_joint: type fixed, parent left_ankle_roll_link, child left_foot_upper_right, origin xyz=0.12 -0.03 -0.03 rpy=0 0 0
- added joint right_foot_line_contact_lower_fix_joint: type fixed, parent right_ankle_roll_link, child right_foot_line_contact_lower, origin xyz=-0.05 0.0 -0.03 rpy=0 0 0
- added joint right_foot_line_contact_upper_fix_joint: type fixed, parent right_ankle_roll_link, child right_foot_line_contact_upper, origin xyz=0.12 0.0 -0.03 rpy=0 0 0
- added joint right_foot_lower_left_fix_joint: type fixed, parent right_ankle_roll_link, child right_foot_lower_left, origin xyz=-0.05 0.025 -0.03 rpy=0 0 0
- added joint right_foot_lower_right_fix_joint: type fixed, parent right_ankle_roll_link, child right_foot_lower_right, origin xyz=-0.05 -0.025 -0.03 rpy=0 0 0
- added joint right_foot_point_contact_fix_joint: type fixed, parent right_ankle_roll_link, child right_foot_point_contact, origin xyz=0.0 0.0 -0.03 rpy=0 0 0
- added joint right_foot_upper_left_fix_joint: type fixed, parent right_ankle_roll_link, child right_foot_upper_left, origin xyz=0.12 0.03 -0.03 rpy=0 0 0
- added joint right_foot_upper_right_fix_joint: type fixed, parent right_ankle_roll_link, child right_foot_upper_right, origin xyz=0.12 -0.03 -0.03 rpy=0 0 0

Commit message: Add contact frames on the palms

File: robots/g1_description/g1_23dof.urdf (robot description, URDF)
Before this commit: robot g1_23dof, 46 links, 45 joints
Links:
- added link left_hand_point_contact
- added link right_hand_point_contact
Joints:
- added joint left_hand_point_contact_fix_joint: type fixed, parent left_wrist_roll_rubber_hand, child left_hand_point_contact, origin xyz=0.17 0.0 0.0 rpy=0 0 0
- added joint right_hand_point_contact_fix_joint: type fixed, parent right_wrist_roll_rubber_hand, child right_hand_point_contact, origin xyz=0.17 0.0 0.0 rpy=0 0 0

Commit message: Add floating dummy frame

File: robots/g1_description/g1_23dof.urdf (robot description, URDF)
Before this commit: robot g1_23dof, 48 links, 47 joints
Links:
- added link world
Joints:
- added joint dummy: type floating, parent world, child pelvis, origin xyz=0.0 0.0 -0.03 rpy=0 0 0
