Commit message: Update 29 dof model with contact frames

File: robots/g1_description/g1_29dof.urdf (robot description, URDF)
Before this commit: robot g1_29dof, 39 links, 38 joints
Links:
- added link left_foot_line_contact_lower
- added link left_foot_line_contact_upper
- added link left_foot_lower_left
- added link left_foot_lower_right
- added link left_foot_point_contact
- added link left_foot_upper_left
- added link left_foot_upper_right
- added link left_hand_point_contact
- added link right_foot_line_contact_lower
- added link right_foot_line_contact_upper
- added link right_foot_lower_left
- added link right_foot_lower_right
- added link right_foot_point_contact
- added link right_foot_upper_left
- added link right_foot_upper_right
- added link right_hand_point_contact
- added link world
Joints:
- added joint dummy: type floating, parent world, child pelvis, origin xyz=0.0 0.0 -0.03 rpy=0 0 0
- added joint left_foot_line_contact_lower_fix_joint: type fixed, parent left_ankle_roll_link, child left_foot_line_contact_lower, origin xyz=-0.05 0.0 -0.03 rpy=0 0 0
- added joint left_foot_line_contact_upper_fix_joint: type fixed, parent left_ankle_roll_link, child left_foot_line_contact_upper, origin xyz=0.12 0.0 -0.03 rpy=0 0 0
- added joint left_foot_lower_left_fix_joint: type fixed, parent left_ankle_roll_link, child left_foot_lower_left, origin xyz=-0.05 0.025 -0.03 rpy=0 0 0
- added joint left_foot_lower_right_fix_joint: type fixed, parent left_ankle_roll_link, child left_foot_lower_right, origin xyz=-0.05 -0.025 -0.03 rpy=0 0 0
- added joint left_foot_point_contact_fix_joint: type fixed, parent left_ankle_roll_link, child left_foot_point_contact, origin xyz=0.0 0.0 -0.03 rpy=0 0 0
- added joint left_foot_upper_left_fix_joint: type fixed, parent left_ankle_roll_link, child left_foot_upper_left, origin xyz=0.12 0.03 -0.03 rpy=0 0 0
- added joint left_foot_upper_right_fix_joint: type fixed, parent left_ankle_roll_link, child left_foot_upper_right, origin xyz=0.12 -0.03 -0.03 rpy=0 0 0
- added joint left_hand_point_contact_fix_joint: type fixed, parent left_rubber_hand, child left_hand_point_contact, origin xyz=0.17 0.0 0.0 rpy=0 0 0
- added joint right_foot_line_contact_lower_fix_joint: type fixed, parent right_ankle_roll_link, child right_foot_line_contact_lower, origin xyz=-0.05 0.0 -0.03 rpy=0 0 0
- added joint right_foot_line_contact_upper_fix_joint: type fixed, parent right_ankle_roll_link, child right_foot_line_contact_upper, origin xyz=0.12 0.0 -0.03 rpy=0 0 0
- added joint right_foot_lower_left_fix_joint: type fixed, parent right_ankle_roll_link, child right_foot_lower_left, origin xyz=-0.05 0.025 -0.03 rpy=0 0 0
- added joint right_foot_lower_right_fix_joint: type fixed, parent right_ankle_roll_link, child right_foot_lower_right, origin xyz=-0.05 -0.025 -0.03 rpy=0 0 0
- added joint right_foot_point_contact_fix_joint: type fixed, parent right_ankle_roll_link, child right_foot_point_contact, origin xyz=0.0 0.0 -0.03 rpy=0 0 0
- added joint right_foot_upper_left_fix_joint: type fixed, parent right_ankle_roll_link, child right_foot_upper_left, origin xyz=0.12 0.03 -0.03 rpy=0 0 0
- added joint right_foot_upper_right_fix_joint: type fixed, parent right_ankle_roll_link, child right_foot_upper_right, origin xyz=0.12 -0.03 -0.03 rpy=0 0 0
- added joint right_hand_point_contact_fix_joint: type fixed, parent right_rubber_hand, child right_hand_point_contact, origin xyz=0.17 0.0 0.0 rpy=0 0 0
